Commit message: [robots/kortex_robot.xacro] Fix joint definition to support multiple arms

File: kortex_description/robots/kortex_robot.xacro (robot description, xacro)
@@ -1,5 +1,5 @@
 <?xml version="1.0"?>
 <robot xmlns:xacro="http://ros.org/wiki/xacro">
-    <xacro:macro name="load_robot" params="arm gripper dof vision sim prefix">
+    <xacro:macro name="load_robot" params="arm gripper dof vision sim prefix parent_link:=world">
         <!-- Files to include -->
         <xacro:include filename="$(find kortex_description)/arms/${arm}/${dof}dof/urdf/${arm}_macro.xacro" />
@@ -16,13 +16,9 @@
         </xacro:if>
         <!-- Run the macros -->
-        <!-- For gazebo-->
-        <xacro:if value="${sim}">
-            <link name="world" />
-            <joint name="world_to_root" type="fixed">
-                <child link="${prefix}base_link" />
-                <parent link="world" />
-                <origin xyz="0 0 0" rpy="0 0 0" />
-            </joint>
-        </xacro:if>
+        <joint name="${prefix}_base_joint" type="fixed">
+            <child link="${prefix}_base_link" />
+            <parent link="${parent_link}" />
+            <origin xyz="0 0 0" rpy="0 0 0" />
+        </joint>
         <!-- Load the arm -->
         <xacro:load_arm parent="" dof="${dof}" vision="${vision}" prefix="${prefix}">
